File: Venom.kicad_pcb (KiCad board)
At the start: 2 copper layers, 72 x 42 mm, 15 parts, among them CN1 HC-XH-5A-G, CN2 HC-PH-8A-G, CN3 HC-XH-8A-G, CN4 HC-XH-8A-G, CN5 HC-XH-2A-G, CN6 HC-PH-7A-G, SW1 GT-TC030A-H020-L1N, SW2 GT-TC030A-H020-L1N, U1 Pico

Commit message: WIP embedded design
Parts:
- added C1: 1u, Capacitor_SMD:C_0402_1005Metric, F.Cu at (140.3, 104.3)
- added C10: 1u, Capacitor_SMD:C_0402_1005Metric, F.Cu at (132.3, 100.2)
- added C11: 100n, Capacitor_SMD:C_0402_1005Metric, F.Cu at (129.9, 90.9)
- added C12: 100n, Capacitor_SMD:C_0402_1005Metric, F.Cu at (109.7, 105.0)
- added C13: 100n, Capacitor_SMD:C_0402_1005Metric, F.Cu at (112.6, 99.1)
- added C14: 100n, Capacitor_SMD:C_0402_1005Metric, F.Cu at (112.6, 101.0)
- added C15: 100n, Capacitor_SMD:C_0402_1005Metric, F.Cu at (129.6, 101.6)
- added C16: 100n, Capacitor_SMD:C_0402_1005Metric, F.Cu at (130.6, 101.6)
- added C2: 30p, Capacitor_SMD:C_0402_1005Metric, F.Cu at (104.0, 101.0)
- added C3: 30p, Capacitor_SMD:C_0402_1005Metric, F.Cu at (104.0, 103.0)
- added C4: 1u, Capacitor_SMD:C_0402_1005Metric, F.Cu at (135.2, 104.3)
- added C5: 100n, Capacitor_SMD:C_0402_1005Metric, F.Cu at (140.5, 91.6)
- added C6: 100n, Capacitor_SMD:C_0402_1005Metric, F.Cu at (136.1, 94.9)
- added C7: 100n, Capacitor_SMD:C_0402_1005Metric, F.Cu at (106.8, 103.0)
- added C8: 1u, Capacitor_SMD:C_0402_1005Metric, F.Cu at (133.4, 99.2)
- added C9: 100n, Capacitor_SMD:C_0402_1005Metric, F.Cu at (133.4, 96.0)
- added R6: 5.1k, Resistor_SMD:R_0402_1005Metric, F.Cu at (141.2, 96.4)
- added R7: 5.1k, Resistor_SMD:R_0402_1005Metric, F.Cu at (140.7, 100.4)
- added SW3: GT-TC030A-H020-L1N, easyeda2kicad:SW-SMD_4P-L3.6-W3.0-P1.50-LS4.7, F.Cu at (146.6, 84.7)
- added U2: W25Q128JVS, Package_SO:SOIC-8_5.23x5.23mm_P1.27mm, F.Cu at (136.9, 87.9)
- added U3: RP2040, RP2040:RP2040-QFN-56, F.Cu at (126.7, 96.2)
- added USB1: HRO-TYPE-C-31-M-12, Type-C:HRO-TYPE-C-31-M-12-Assembly, F.Cu at (150.8, 99.1)
- added Y1: Crystal_GND24, Crystal:Crystal_SMD_3225-4Pin_3.2x2.5mm, F.Cu at (92.5, 92.3)
- R1, R5: value 0603WAF3300T5E -> 1k; footprint easyeda2kicad:R0603 -> Resistor_SMD:R_0402_1005Metric
- R2: value 0603WAF3300T5E -> 10k; footprint easyeda2kicad:R0603 -> Resistor_SMD:R_0402_1005Metric
- R3, R4: value 0603WAF3300T5E -> 27; footprint easyeda2kicad:R0603 -> Resistor_SMD:R_0402_1005Metric
- U1: value Pico -> TLV73333PDBV; footprint MCU_RaspberryPi_and_Boards:RPi_Pico_SMD_TH -> Package_TO_SOT_SMD:SOT-23-5
- moved SW2 65.5 mm to (146.6, 89.6)
- moved R1 31.1 mm to (141.4, 84.0), turned to 0 degrees
- moved R2 30.3 mm to (141.4, 85.0), turned to 180 degrees
- moved R5 26.9 mm to (116.8, 92.0)
- moved R3 18.0 mm to (133.4, 97.1), turned to 180 degrees
- moved R4 16.9 mm to (133.4, 98.1), turned to 180 degrees
- moved U1 16.6 mm to (137.8, 103.8), turned to 180 degrees
- moved OSHW1 10.1 mm to (82.0, 104.0)
Connections:
- R1 pad 1: PLEDR1 -> QSPI_SS
- R1 pad 2: PLED 1 -> BOOTSEL
- R2 pad 1: PLEDR2 -> +3V3
- R2 pad 2: PLED 2 -> QSPI_SS
- R3 pad 1: PLEDR3 -> D+
- R3 pad 2: PLED 3 -> Net-(U3-USB_DP)
- R4 pad 1: PLEDR4 -> D-
- R4 pad 2: PLED 4 -> Net-(U3-USB_DM)
- R5 pad 1: TLEDR1 -> Net-(C3-Pad1)
- R5 pad 2: TURBO LED -> XOUT
- U1 pad 1: PS4 MODE -> +5V
- U1 pad 2: TURBO1 -> GND
- U1 pad 3: unconnected-(U1-GND-Pad3) -> +5V
- U1 pad 4: UP -> unconnected-(U1-NC-Pad4)
- U1 pad 5: DOWN -> +3V3
Routing:
- net RUN: track 92.7 -> 27.8 mm, vias 0 -> 2
- net UP: track 54.3 -> 0.00 mm
- net RIGHT: track 54.1 -> 0.00 mm
- net DOWN: track 53.7 -> 0.00 mm
- net TURBO: track 53.1 -> 0.00 mm
- net LEFT: track 52.5 -> 0.00 mm
- net +3V3: track 0.00 -> 49.3 mm, vias 0 -> 2
- net TURBO1: track 41.0 -> 0.00 mm
- net PS4 MODE: track 40.9 -> 0.00 mm
- net S2 (START): track 36.9 -> 0.00 mm
- net PLEDR1: track 28.0 -> 0.00 mm
- net PLEDR2: track 24.8 -> 0.00 mm
- net TLEDR1: track 22.7 -> 0.00 mm
- net GND: track 6.32 -> 27.9 mm, vias 3 -> 15
- net +5V: track 0.00 -> 20.8 mm
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- added copper zone on F.Cu, net GND
Other:
- board text added: "BOOT"
- board text added: "USB1"
- board text removed: "JLCJLCJLCJLC"
